Commit message: D435 深度体素接入与 PCL 离群点影子对照
- 独立 B Costmap 静止标障/清障：中央、左、右低盒各有有效样本
- 新增 PCL RadiusOutlierRemoval 影子节点（手动启动、不接管地图）
- 操作手册新增第 30.9/30.10 节；RViz 增加绿色影子预览
- bao 主机 RViz 联调、深度灰度图显示、Fast DDS 域 31 跨机通信
- 测试记录 R13 位置修正；15 项 carcar_camera 测试全部通过
- 黄色体素偶现空地闪烁散点，根因待定位（缺逐帧蓝点/二维格证据）

File: src/carcar_description/urdf/carcar.urdf.xacro (robot description, xacro)
@@ -5,4 +5,10 @@
     本文件只负责组装；已确认值和待实测值集中维护在 carcar_dimensions.xacro。
   -->
+  <xacro:arg name="camera_extrinsics_file"
+    default="$(find carcar_description)/config/camera_extrinsics.yaml"/>
+  <!-- 可动关节仅用于静止调试；当前 /joint_states 相机角为命令估计，无反馈。 -->
+  <xacro:arg name="camera_tilt_dynamic" default="false"/>
+  <xacro:property name="camera_extrinsics"
+    value="${xacro.load_yaml('$(arg camera_extrinsics_file)')}"/>
   <xacro:include filename="carcar_dimensions.xacro"/>
   <xacro:include filename="carcar_materials.xacro"/>

File: src/carcar_description/urdf/carcar_chassis.xacro (robot description, xacro)
@@ -99,5 +99,5 @@
       <visual name="upper_structure_mesh">
         <origin
-          xyz="${overall_rear_x} 0.065 ${ground_clearance - wheel_radius - upper_deck_z}"
+          xyz="${overall_rear_x} 0.065 ${upper_deck_top_height - wheel_radius - upper_deck_z - 0.130}"
           rpy="${pi / 2} 0 0"/>
         <geometry>

File: src/carcar_description/urdf/carcar_dimensions.xacro (robot description, xacro)
@@ -13,6 +13,6 @@
   <xacro:property name="overall_height" value="0.230"/>
   <xacro:property name="ground_clearance" value="0.010"/>
-  <!-- 相机镜头面为当前最前端；据整车总长反推最后端 X=-0.105 m，待包络复测时核对。 -->
-  <xacro:property name="overall_front_x" value="${camera_x}"/>
+  <!-- 相机安装外参与车身包络解耦；标定结果变化不得改变已测整车尺寸。 -->
+  <xacro:property name="overall_front_x" value="0.130"/>
   <xacro:property name="overall_rear_x" value="${overall_front_x - overall_length}"/>
   <!-- ======================== 厂家机械资料，不是安装外参 ================== -->
@@ -40,9 +40,9 @@
   <xacro:property name="motor_length" value="0.050"/>
   <xacro:property name="chassis_standoff_radius" value="0.003"/>
-  <!-- 蓝色顶板为实测值；顶面离地 140 mm，以下换算为相对 base_link 的板中心。 -->
+  <!-- 2026-09-23 用户复核蓝色顶板顶面离地 135 mm；以下换算为板中心。 -->
   <xacro:property name="upper_deck_x" value="0.220"/>
   <xacro:property name="upper_deck_y" value="0.130"/>
   <xacro:property name="upper_deck_thickness" value="0.010"/>
-  <xacro:property name="upper_deck_top_height" value="0.140"/>
+  <xacro:property name="upper_deck_top_height" value="0.135"/>
   <xacro:property name="upper_deck_z"
     value="${upper_deck_top_height - wheel_radius - upper_deck_thickness / 2}"/>
@@ -65,10 +65,27 @@
   <xacro:property name="laser_xyz" value="-0.050 0 ${0.217 - wheel_radius}"/>
   <xacro:property name="laser_rpy" value="0 0 0"/>
-  <!-- RealSense 左红外中心由用户相对 base_footprint 实测；实机图像确认相机倒装。 -->
-  <xacro:property name="camera_x" value="0.130"/>
-  <xacro:property name="camera_y" value="0.033"/>
-  <xacro:property name="camera_z" value="${0.170 - wheel_radius}"/>
+  <!-- RealSense 安装外参从独立 YAML 读取；默认文件仍是尺量初值，待 TF-005 标定验收。 -->
+  <xacro:property name="camera_x" value="${camera_extrinsics['translation']['x']}"/>
+  <xacro:property name="camera_y" value="${camera_extrinsics['translation']['y']}"/>
+  <xacro:property name="camera_z" value="${camera_extrinsics['translation']['z']}"/>
   <xacro:property name="camera_xyz" value="${camera_x} ${camera_y} ${camera_z}"/>
-  <xacro:property name="camera_rpy" value="${pi} 0 0"/>
+  <xacro:property name="camera_rpy"
+    value="${camera_extrinsics['rpy']['roll']} ${camera_extrinsics['rpy']['pitch']} ${camera_extrinsics['rpy']['yaw']}"/>
+  <!-- 2026-09-23 用户复核粗量输出轴中心=(90,0,145) mm，相对 base_footprint。 -->
+  <xacro:property name="camera_tilt_pivot_x" value="0.090"/>
+  <xacro:property name="camera_tilt_pivot_y" value="0.000"/>
+  <xacro:property name="camera_tilt_pivot_z" value="${0.145 - wheel_radius}"/>
+  <xacro:property name="camera_tilt_pivot_xyz"
+    value="${camera_tilt_pivot_x} ${camera_tilt_pivot_y} ${camera_tilt_pivot_z}"/>
+  <!-- 用户粗量舵机盒质心=(82,-30,145) mm，相对 base_footprint；壳体中心暂按质心放置。 -->
+  <xacro:property name="camera_servo_center_x" value="0.082"/>
+  <xacro:property name="camera_servo_center_y" value="-0.030"/>
+  <xacro:property name="camera_servo_center_z" value="${0.145 - wheel_radius}"/>
+  <xacro:property name="camera_servo_center_in_mount_xyz"
+    value="${camera_servo_center_x - camera_tilt_pivot_x} ${camera_servo_center_y - camera_tilt_pivot_y} ${camera_servo_center_z - camera_tilt_pivot_z}"/>
+  <!-- 视觉近似：照片中的 20KG 级舵机型号和实际包络均待实测。 -->
+  <xacro:property name="camera_servo_body_x" value="0.040"/>
+  <xacro:property name="camera_servo_body_y" value="0.040"/>
+  <xacro:property name="camera_servo_body_z" value="0.020"/>
   <!--
     车体碰撞体到蓝色顶板顶面；传感器另有独立 collision。Nav2 footprint 使用整车

File: src/carcar_description/urdf/carcar_materials.xacro (robot description, xacro)
@@ -6,4 +6,7 @@
   <material name="metal_dark"><color rgba="0.22 0.24 0.27 1.0"/></material>
   <material name="plastic_black"><color rgba="0.035 0.045 0.055 1.0"/></material>
+  <material name="mount_orange"><color rgba="0.95 0.30 0.015 1.0"/></material>
+  <material name="servo_label_pink"><color rgba="0.73 0.13 0.39 1.0"/></material>
+  <material name="servo_case_pink"><color rgba="0.95 0.32 0.57 1.0"/></material>
   <material name="plastic_white"><color rgba="0.91 0.92 0.93 1.0"/></material>
   <material name="wheel_white"><color rgba="0.94 0.94 0.94 1.0"/></material>

File: src/carcar_description/urdf/carcar_sensors.xacro (robot description, xacro)
@@ -10,7 +10,7 @@
   <xacro:macro name="lidar_standoff" params="name x y">
     <visual name="${name}">
-      <origin xyz="${x} ${y} -0.0545" rpy="0 0 0"/>
-      <geometry><cylinder radius="0.003" length="0.035"/></geometry>
-      <material name="plastic_white"/>
+      <origin xyz="${x} ${y} -0.060" rpy="0 0 0"/>
+      <geometry><cylinder radius="0.003" length="0.034"/></geometry>
+      <material name="body_blue"/>
     </visual>
   </xacro:macro>
@@ -38,11 +38,11 @@
     <link name="laser_frame">
       <visual name="lidar_bottom_plate">
-        <origin xyz="0 0 -0.034" rpy="0 0 0"/>
+        <origin xyz="0 0 -0.040" rpy="0 0 0"/>
         <geometry><box size="${lidar_body_x} ${lidar_body_y} 0.006"/></geometry>
         <material name="plastic_black"/>
       </visual>
       <visual name="lidar_fixed_base">
-        <origin xyz="0 0 -0.023" rpy="0 0 0"/>
-        <geometry><cylinder radius="0.044" length="0.016"/></geometry>
+        <origin xyz="0 0 -0.026" rpy="0 0 0"/>
+        <geometry><cylinder radius="0.044" length="0.022"/></geometry>
         <material name="plastic_black"/>
       </visual>
@@ -58,5 +58,6 @@
       </visual>
       <visual name="lidar_mount_plate_mesh">
-        <origin xyz="${overall_rear_x + 0.050} 0.03475 -0.07705" rpy="${pi / 2} 0 0"/>
+        <!-- STL 厚 5 mm；底面落在用户量得离地 135 mm 的蓝色顶板顶面。 -->
+        <origin xyz="${overall_rear_x + 0.050} 0.03475 -0.08205" rpy="${pi / 2} 0 0"/>
         <geometry>
           <mesh filename="package://carcar_description/meshes/vehicle/lidar_mount_plate.stl"
@@ -70,70 +71,131 @@
       <xacro:lidar_standoff name="lidar_rear_right_standoff" x="-0.026" y="-0.033"/>
       <collision name="lidar_collision">
-        <origin xyz="0 0 ${overall_height - 0.217 - lidar_body_z / 2}" rpy="0 0 0"/>
-        <geometry><cylinder radius="0.049" length="${lidar_body_z}"/></geometry>
+        <origin xyz="0 0 -0.015" rpy="0 0 0"/>
+        <geometry><cylinder radius="0.049" length="0.056"/></geometry>
       </collision>
       <collision name="lidar_mount_collision">
-        <origin xyz="${overall_rear_x + 0.082 + 0.050} 0 -0.0745"/>
+        <origin xyz="${overall_rear_x + 0.082 + 0.050} 0 -0.0795"/>
         <geometry><box size="0.164 0.0695 0.005"/></geometry>
       </collision>
     </link>
-    <!--
-      camera_link 位于左红外相机（Infra1）光学中心，是 RealSense 驱动内部 TF 树的
-      安装根。这里只发布 base_link 到 camera_link；camera_*_optical_frame 由
-      realsense-ros 唯一发布。
-    -->
-    <joint name="camera_joint" type="fixed">
-      <parent link="base_link"/>
-      <child link="camera_link"/>
-      <origin xyz="${camera_xyz}" rpy="${camera_rpy}"/>
-    </joint>
-    <link name="camera_link">
-      <visual name="camera_silver_shell">
-        <origin xyz="${-camera_body_x / 2} -0.025 0" rpy="0 0 0"/>
-        <geometry><box size="${camera_body_x} ${camera_body_y} ${camera_body_z}"/></geometry>
-        <material name="plastic_white"/>
-      </visual>
-      <visual name="camera_front_mask">
-        <origin xyz="-0.0005 -0.025 0" rpy="0 0 0"/>
-        <geometry><box size="0.001 0.082 0.018"/></geometry>
-        <material name="plastic_black"/>
-      </visual>
-      <xacro:camera_aperture name="camera_left_ir" y="0" radius="0.006" material="lens_dark"/>
-      <xacro:camera_aperture name="camera_projector" y="-0.017" radius="0.005" material="lens_blue"/>
-      <xacro:camera_aperture name="camera_rgb" y="-0.033" radius="0.006" material="lens_blue"/>
-      <xacro:camera_aperture name="camera_right_ir" y="-0.050" radius="0.006" material="lens_dark"/>
-      <collision name="camera_collision">
-        <origin xyz="${-camera_body_x / 2} -0.025 0" rpy="0 0 0"/>
-        <geometry><box size="${camera_body_x} ${camera_body_y} ${camera_body_z}"/></geometry>
-      </collision>
-    </link>
-    <!-- 支架固定在车体上，不随 camera_link 的 180° 倒装坐标旋转。 -->
+    <!-- 橙色底板锁件和舵机壳固定在车体；轴心坐标为用户粗量值。 -->
     <joint name="camera_mount_joint" type="fixed">
       <parent link="base_link"/>
       <child link="camera_mount_link"/>
-      <origin xyz="${camera_xyz}" rpy="0 0 0"/>
+      <origin xyz="${camera_tilt_pivot_xyz}" rpy="0 0 0"/>
     </joint>
     <link name="camera_mount_link">
-      <visual name="camera_lower_mount_mesh">
-        <!-- 原 X 为横向、Y 为高度、Z 为纵向；底面落在实测顶板上。 -->
-        <origin xyz="-0.105 -0.0675 -0.030" rpy="${pi / 2} 0 ${pi / 2}"/>
-        <geometry>
-          <mesh filename="package://carcar_description/meshes/vehicle/camera_lower_mount.stl"
-            scale="0.001 0.001 0.001"/>
-        </geometry>
-        <material name="body_blue"/>
-      </visual>
-      <visual name="camera_direct_mount_mesh">
-        <!-- 封闭安装端朝相机后壳，长臂沿 -X 伸向底座。 -->
-        <origin xyz="-0.025 -0.066571 -0.026049" rpy="${pi / 2} 0 ${pi}"/>
-        <geometry>
-          <mesh filename="package://carcar_description/meshes/vehicle/camera_direct_mount.stl"
-            scale="0.001 0.001 0.001"/>
-        </geometry>
-        <material name="body_blue"/>
-      </visual>
-      <collision name="camera_mount_collision">
-        <origin xyz="-0.0675 -0.033 0"/>
-        <geometry><box size="0.085 0.069 0.060"/></geometry>
+      <visual name="camera_servo_case">
+        <origin xyz="${camera_servo_center_in_mount_xyz}" rpy="0 0 0"/>
+        <geometry><box size="${camera_servo_body_x} ${camera_servo_body_y} ${camera_servo_body_z}"/></geometry>
+        <material name="servo_case_pink"/>
+      </visual>
+      <visual name="camera_servo_label">
+        <origin xyz="${camera_servo_center_x - camera_tilt_pivot_x} ${camera_servo_center_y - camera_tilt_pivot_y} ${camera_servo_center_z - camera_tilt_pivot_z + camera_servo_body_z / 2 + 0.0005}" rpy="0 0 0"/>
+        <geometry><box size="0.032 0.026 0.001"/></geometry>
+        <material name="servo_label_pink"/>
+      </visual>
+      <visual name="camera_servo_horn">
+        <origin xyz="0 -0.005 0" rpy="${pi / 2} 0 0"/>
+        <geometry><cylinder radius="0.008" length="0.010"/></geometry>
+        <material name="metal_silver"/>
+      </visual>
+      <collision name="camera_servo_collision">
+        <origin xyz="${camera_servo_center_in_mount_xyz}" rpy="0 0 0"/>
+        <geometry><box size="${camera_servo_body_x} ${camera_servo_body_y} ${camera_servo_body_z}"/></geometry>
+      </collision>
+    </link>
+    <!-- 两个橙色锁件固定在舵机前后端，双孔沿 Y 横排，平底贴在顶板上。 -->
+    <joint name="camera_servo_left_foot_joint" type="fixed">
+      <parent link="camera_mount_link"/>
+      <child link="camera_servo_left_foot_link"/>
+      <!-- 后端：X=52..62 mm，竖边贴近舵机盒后端 X=62 mm。 -->
+      <origin xyz="-0.038 0.015392723 -0.010" rpy="${pi / 2} 0 0"/>
+    </joint>
+    <link name="camera_servo_left_foot_link">
+      <visual name="camera_servo_left_foot">
+        <geometry><mesh filename="package://carcar_description/meshes/vehicle/camera_servo_left_foot.stl"
+          scale="0.001 0.001 0.001"/></geometry>
+        <material name="mount_orange"/>
+      </visual>
+      <collision name="camera_servo_left_foot_collision">
+        <origin xyz="0.005 0.00995 0.045392723" rpy="0 0 0"/>
+        <geometry><box size="0.010 0.0199 0.020"/></geometry>
+      </collision>
+    </link>
+    <joint name="camera_servo_right_foot_joint" type="fixed">
+      <parent link="camera_mount_link"/>
+      <child link="camera_servo_right_foot_link"/>
+      <!-- 前端锁件绕自身中心的车体 Z 轴翻转 180°；外廓仍为 X=102..112、Y=-40..-20 mm。 -->
+      <origin xyz="0.012 0.015392723 -0.010" rpy="${pi / 2} 0 0"/>
+    </joint>
+    <link name="camera_servo_right_foot_link">
+      <visual name="camera_servo_right_foot">
+        <geometry><mesh filename="package://carcar_description/meshes/vehicle/camera_servo_right_foot.stl"
+          scale="0.001 0.001 0.001"/></geometry>
+        <material name="mount_orange"/>
+      </visual>
+      <collision name="camera_servo_right_foot_collision">
+        <origin xyz="0.005 0.00995 0.045392723" rpy="0 0 0"/>
+        <geometry><box size="0.010 0.0199 0.020"/></geometry>
+      </collision>
+    </link>
+    <!-- 正式导航固定平视；可动模式仅用于静止命令估计调试，不代表角度反馈。 -->
+    <xacro:if value="$(arg camera_tilt_dynamic)">
+      <joint name="camera_tilt_joint" type="revolute">
+        <parent link="camera_mount_link"/>
+        <child link="camera_tilt_link"/>
+        <origin xyz="0 0 0" rpy="0 0 0"/>
+        <axis xyz="0 1 0"/>
+        <limit lower="${(85.0 - 140.5) * pi / 180.0}"
+          upper="${(160.0 - 140.5) * pi / 180.0}" effort="1.0" velocity="1.0"/>
+      </joint>
+    </xacro:if>
+    <xacro:unless value="$(arg camera_tilt_dynamic)">
+      <joint name="camera_tilt_joint" type="fixed">
+        <parent link="camera_mount_link"/>
+        <child link="camera_tilt_link"/>
+        <origin xyz="0 0 0" rpy="0 0 0"/>
+      </joint>
+    </xacro:unless>
+    <link name="camera_tilt_link">
+      <visual name="camera_tilt_bracket">
+        <!-- STL 小 X 端为舵机轴孔（约 9,35,8.5 mm），大 X 端为相机安装面。 -->
+        <origin xyz="-0.009 -0.035 -0.0085" rpy="0 0 0"/>
+        <geometry><mesh filename="package://carcar_description/meshes/vehicle/camera_tilt_bracket.stl"
+          scale="0.001 0.001 0.001"/></geometry>
+        <material name="plastic_black"/>
+      </visual>
+      <collision name="camera_tilt_bracket_collision">
+        <origin xyz="0.0115 0 0.005" rpy="0 0 0"/>
+        <geometry><box size="0.043 0.072 0.030"/></geometry>
+      </collision>
+    </link>
+    <!-- camera_link 是 RealSense 左红外光心；候选 YAML 保持中位时 base_link 外参语义。 -->
+    <joint name="camera_joint" type="fixed">
+      <parent link="camera_tilt_link"/>
+      <child link="camera_link"/>
+      <origin xyz="${camera_x - camera_tilt_pivot_x} ${camera_y - camera_tilt_pivot_y} ${camera_z - camera_tilt_pivot_z}"
+        rpy="${camera_rpy}"/>
+    </joint>
+    <link name="camera_link">
+      <visual name="camera_silver_shell">
+        <origin xyz="${-camera_body_x / 2} -0.0175 0" rpy="0 0 0"/>
+        <geometry><box size="${camera_body_x} ${camera_body_y} ${camera_body_z}"/></geometry>
+        <material name="plastic_white"/>
+      </visual>
+      <visual name="camera_front_mask">
+        <origin xyz="-0.0005 -0.0175 0" rpy="0 0 0"/>
+        <geometry><box size="0.001 0.082 0.018"/></geometry>
+        <material name="plastic_black"/>
+      </visual>
+      <!-- 官方 D435 正面左到右：右红外、投射器、左红外、RGB。左红外为深度原点。 -->
+      <xacro:camera_aperture name="camera_left_ir" y="0" radius="0.006" material="lens_dark"/>
+      <xacro:camera_aperture name="camera_projector" y="-0.029" radius="0.008" material="lens_blue"/>
+      <xacro:camera_aperture name="camera_rgb" y="0.015" radius="0.005" material="lens_blue"/>
+      <xacro:camera_aperture name="camera_right_ir" y="-0.050" radius="0.006" material="lens_dark"/>
+      <collision name="camera_collision">
+        <origin xyz="${-camera_body_x / 2} -0.0175 0" rpy="0 0 0"/>
+        <geometry><box size="${camera_body_x} ${camera_body_y} ${camera_body_z}"/></geometry>
       </collision>
     </link>
